File: heatbed_pcb/bed.brd (EAGLE design)
At the start: 34 x 32 mm, 0 parts

Commit message: .
Routing:
- net S$9: track 352.5 -> 257.9 mm
- net S$25: track 0.00 -> 92.2 mm
- net S$18: track 352.5 -> 348.8 mm
- net S$26: track 0.00 -> 1.35 mm
- net S$30: track 0.00 -> 1.05 mm
- net S$27: track 0.00 -> 1.05 mm
- net S$28: track 0.00 -> 0.73 mm
- net S$29: track 0.00 -> 0.68 mm
Changed lines of the file:
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@@
 <wire x1="33" y1="13.125" x2="0.75" y2="13.125" width="0.2" layer="1"/>
+</signal>
+<signal name="S$23">
+<wire x1="0.75" y1="15.625" x2="0.75" y2="15.875" width="0.2" layer="1"/>
+</signal>
+<signal name="S$24">
+<wire x1="31.8" y1="15.375" x2="31.8" y2="15.625" width="0.2" layer="1"/>
 </signal>
 <signal name="S$9">
@@
 <wire x1="31.8" y1="15.125" x2="0.75" y2="15.125" width="0.2" layer="1"/>
 <wire x1="0.75" y1="15.125" x2="0.75" y2="15.375" width="0.2" layer="1"/>
-<wire x1="0.75" y1="15.375" x2="31.8" y2="15.375" width="0.2" layer="1"/>
-<wire x1="31.8" y1="15.375" x2="31.8" y2="15.625" width="0.2" layer="1"/>
-<wire x1="31.8" y1="15.625" x2="0.75" y2="15.625" width="0.2" layer="1"/>
-<wire x1="0.75" y1="15.625" x2="0.75" y2="15.875" width="0.2" layer="1"/>
-<wire x1="0.75" y1="15.875" x2="32.75" y2="15.875" width="0.2" layer="1"/>
 </signal>
 <signal name="S$10">
@@
 <wire x1="33" y1="18.875" x2="0.75" y2="18.875" width="0.2" layer="1"/>
 </signal>
+<signal name="S$22">
+<wire x1="31.8" y1="16.625" x2="31.8" y2="16.375" width="0.2" layer="1"/>
+</signal>
+<signal name="S$21">
+<wire x1="0.75" y1="16.375" x2="0.75" y2="16.125" width="0.2" layer="1"/>
+</signal>
 <signal name="S$18">
 <wire x1="0.75" y1="18.875" x2="0.75" y2="18.625" width="0.2" layer="1"/>
@@
 <wire x1="31.8" y1="16.875" x2="0.75" y2="16.875" width="0.2" layer="1"/>
 <wire x1="0.75" y1="16.875" x2="0.75" y2="16.625" width="0.2" layer="1"/>
-<wire x1="0.75" y1="16.625" x2="31.8" y2="16.625" width="0.2" layer="1"/>
-<wire x1="31.8" y1="16.625" x2="31.8" y2="16.375" width="0.2" layer="1"/>
-<wire x1="31.8" y1="16.375" x2="0.75" y2="16.375" width="0.2" layer="1"/>
-<wire x1="0.75" y1="16.375" x2="0.75" y2="16.125" width="0.2" layer="1"/>
-<wire x1="0.75" y1="16.125" x2="32.75" y2="16.125" width="0.2" layer="1"/>
+<wire x1="16.4" y1="16.625" x2="0.75" y2="16.625" width="0.2" layer="1"/>
+<wire x1="16.55" y1="16.375" x2="0.75" y2="16.375" width="0.2" layer="1"/>
+<wire x1="16.75" y1="16.125" x2="0.75" y2="16.125" width="0.2" layer="1"/>
+<wire x1="17.25" y1="16.125" x2="32.15" y2="16.125" width="0.2" layer="1"/>
+<wire x1="17.45" y1="16.375" x2="31.8" y2="16.375" width="0.2" layer="1"/>
+<wire x1="17.6" y1="16.625" x2="31.8" y2="16.625" width="0.2" layer="1"/>
 </signal>
 <signal name="S$19">
@@
 <via x="32.425" y="15.225" extent="1-16" drill="0.01" diameter="0.2" shape="square"/>
 </signal>
+<signal name="S$25">
+<wire x1="16.4" y1="15.375" x2="0.75" y2="15.375" width="0.2" layer="1"/>
+<wire x1="16.55" y1="15.625" x2="0.75" y2="15.625" width="0.2" layer="1"/>
+<wire x1="16.75" y1="15.875" x2="0.75" y2="15.875" width="0.2" layer="1"/>
+<wire x1="17.25" y1="15.875" x2="32.15" y2="15.875" width="0.2" layer="1"/>
+<wire x1="17.45" y1="15.625" x2="31.8" y2="15.625" width="0.2" layer="1"/>
+<wire x1="17.6" y1="15.375" x2="31.8" y2="15.375" width="0.2" layer="1"/>
+<wire x1="16.4" y1="15.375" x2="16.4" y2="15.35" width="0.15" layer="1"/>
+<wire x1="16.4" y1="15.35" x2="17.625" y2="15.35" width="0.15" layer="1"/>
+</signal>
+<signal name="S$26">
+<wire x1="16.4" y1="16.6" x2="16.4" y2="16.65" width="0.15" layer="1"/>
+<wire x1="16.4" y1="16.65" x2="17.65" y2="16.65" width="0.15" layer="1"/>
+<wire x1="17.65" y1="16.65" x2="17.65" y2="16.6" width="0.15" layer="1"/>
+</signal>
+<signal name="S$27">
+<wire x1="16.575" y1="16.35" x2="16.575" y2="16.45" width="0.15" layer="1"/>
+<wire x1="16.575" y1="16.45" x2="17.425" y2="16.45" width="0.15" layer="1"/>
+<wire x1="17.425" y1="16.45" x2="17.425" y2="16.35" width="0.15" layer="1"/>
+</signal>
+<signal name="S$28">
+<wire x1="16.775" y1="16.1" x2="16.775" y2="16.25" width="0.15" layer="1"/>
+<wire x1="16.775" y1="16.25" x2="17.225" y2="16.25" width="0.15" layer="1"/>
+<wire x1="17.225" y1="16.25" x2="17.225" y2="16.125" width="0.15" layer="1"/>
+</signal>
+<signal name="S$29">
+<wire x1="17.225" y1="15.875" x2="17.225" y2="15.75" width="0.15" layer="1"/>
+<wire x1="17.225" y1="15.75" x2="16.775" y2="15.75" width="0.15" layer="1"/>
+<wire x1="16.775" y1="15.75" x2="16.775" y2="15.85" width="0.15" layer="1"/>
+</signal>
+<signal name="S$30">
+<wire x1="16.575" y1="15.65" x2="16.575" y2="15.55" width="0.15" layer="1"/>
+<wire x1="16.575" y1="15.55" x2="17.425" y2="15.55" width="0.15" layer="1"/>
+<wire x1="17.425" y1="15.55" x2="17.425" y2="15.65" width="0.15" layer="1"/>
+</signal>
 </signals>

Commit message: .
Routing:
- net S$31: track 0.00 -> 51.6 mm
- net S$10: track 464.8 -> 414.1 mm
- net S$18: track 348.8 -> 334.4 mm
- net S$32: track 0.00 -> 13.6 mm
- net S$33: track 0.00 -> 1.96 mm
- net S$34: track 0.00 -> 1.51 mm
- net S$1: track 464.8 -> 465.6 mm
Changed lines of the file:
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@@
 <setting verticaltext="up"/>
 </settings>
-<grid distance="0.025" unitdist="mm" unit="mm" style="dots" multiple="5" display="yes" altdistance="0.125" altunitdist="mm" altunit="mm"/>
+<grid distance="0.05" unitdist="mm" unit="mm" style="dots" multiple="5" display="yes" altdistance="0.025" altunitdist="mil" altunit="mil"/>
 <layers>
 <layer number="1" name="Top" color="4" fill="1" visible="yes" active="yes"/>
@@
 <wire x1="32.175" y1="17.2" x2="32.175" y2="14.8" width="0" layer="20"/>
 <hole x="17" y="16" drill="0.3"/>
+<hole x="3" y="0.5" drill="0.3"/>
+<hole x="31" y="31.5" drill="0.3"/>
+<hole x="31" y="0.5" drill="0.3"/>
+<hole x="3" y="31.5" drill="0.3"/>
 </plain>
 <attributes>
@@
 <signals>
 <signal name="S$1">
-<wire x1="33.375" y1="0.625" x2="0.75" y2="0.625" width="0.2" layer="1"/>
-<wire x1="0.75" y1="0.625" x2="0.75" y2="0.875" width="0.2" layer="1"/>
-<wire x1="33.375" y1="0.625" x2="33.375" y2="3.5" width="0.2" layer="1"/>
+<wire x1="33.375" y1="0.175" x2="0.75" y2="0.175" width="0.2" layer="1"/>
+<wire x1="0.75" y1="0.175" x2="0.75" y2="0.875" width="0.2" layer="1"/>
+<wire x1="33.375" y1="0.175" x2="33.375" y2="3.5" width="0.2" layer="1"/>
 <wire x1="33.375" y1="3.5" x2="31.5" y2="3.5" width="0.2" layer="1"/>
 <wire x1="31.5" y1="3.5" x2="31.5" y2="6.5" width="0.2" layer="1"/>
@@
 <wire x1="0.75" y1="15.125" x2="0.75" y2="15.375" width="0.2" layer="1"/>
 </signal>
+<signal name="S$31">
+<wire x1="33.5" y1="25.5" x2="33.5" y2="16.75" width="0.2" layer="1"/>
+<wire x1="31.5" y1="25.5" x2="33.5" y2="25.5" width="0.2" layer="1"/>
+<wire x1="31.5" y1="28.5" x2="31.5" y2="25.5" width="0.2" layer="1"/>
+<wire x1="33.375" y1="28.5" x2="31.5" y2="28.5" width="0.2" layer="1"/>
+<wire x1="33.375" y1="31.825" x2="33.375" y2="28.5" width="0.2" layer="1"/>
+<wire x1="33.375" y1="31.825" x2="0.75" y2="31.825" width="0.2" layer="1"/>
+</signal>
 <signal name="S$10">
-<wire x1="33.375" y1="31.375" x2="0.75" y2="31.375" width="0.2" layer="1"/>
-<wire x1="0.75" y1="31.375" x2="0.75" y2="31.125" width="0.2" layer="1"/>
-<wire x1="33.375" y1="31.375" x2="33.375" y2="28.5" width="0.2" layer="1"/>
-<wire x1="33.375" y1="28.5" x2="31.5" y2="28.5" width="0.2" layer="1"/>
-<wire x1="31.5" y1="28.5" x2="31.5" y2="25.5" width="0.2" layer="1"/>
-<wire x1="31.5" y1="25.5" x2="33.5" y2="25.5" width="0.2" layer="1"/>
 <wire x1="0.75" y1="31.125" x2="33" y2="31.125" width="0.2" layer="1"/>
 <wire x1="33" y1="31.125" x2="33" y2="30.875" width="0.2" layer="1"/>
@@
 <wire x1="2.5" y1="28.125" x2="31.125" y2="28.125" width="0.2" layer="1"/>
 <wire x1="31.125" y1="28.125" x2="31.125" y2="27.875" width="0.2" layer="1"/>
-<wire x1="33.5" y1="25.5" x2="33.5" y2="16.75" width="0.2" layer="1"/>
+<wire x1="0.75" y1="31.825" x2="0.75" y2="31.125" width="0.2" layer="1"/>
 </signal>
 <signal name="S$11">
@@
 </signal>
 <signal name="S$22">
-<wire x1="31.8" y1="16.625" x2="31.8" y2="16.375" width="0.2" layer="1"/>
+<wire x1="24.65" y1="16.625" x2="24.65" y2="16.375" width="0.2" layer="1"/>
 </signal>
 <signal name="S$21">
@@
 <wire x1="16.75" y1="16.125" x2="0.75" y2="16.125" width="0.2" layer="1"/>
 <wire x1="17.25" y1="16.125" x2="32.15" y2="16.125" width="0.2" layer="1"/>
-<wire x1="17.45" y1="16.375" x2="31.8" y2="16.375" width="0.2" layer="1"/>
-<wire x1="17.6" y1="16.625" x2="31.8" y2="16.625" width="0.2" layer="1"/>
+<wire x1="17.45" y1="16.375" x2="24.65" y2="16.375" width="0.2" layer="1"/>
+<wire x1="17.6" y1="16.625" x2="24.65" y2="16.625" width="0.2" layer="1"/>
 </signal>
 <signal name="S$19">
@@
 <signal name="S$20">
 <via x="32.425" y="15.225" extent="1-16" drill="0.01" diameter="0.2" shape="square"/>
+<via x="24.991840625" y="16.386265625" extent="1-16" drill="0.01" diameter="0.2" shape="square"/>
+<via x="24.990521875" y="16.62898125" extent="1-16" drill="0.01" diameter="0.2" shape="square"/>
 </signal>
 <signal name="S$25">
@@
 <wire x1="17.425" y1="15.55" x2="17.425" y2="15.65" width="0.15" layer="1"/>
 </signal>
+<signal name="S$32">
+<wire x1="25.0127" y1="16.40635" x2="31.8627" y2="16.40635" width="0.15" layer="1"/>
+<wire x1="25.0127" y1="16.609525" x2="31.7127" y2="16.609525" width="0.15" layer="1"/>
+</signal>
+<signal name="S$33">
+<wire x1="31.677609375" y1="16.637634375" x2="32.1" y2="16.637634375" width="0.1" layer="1"/>
+<wire x1="32.1" y1="16.637634375" x2="32.1" y2="16.9" width="0.1" layer="1"/>
+<wire x1="32.1" y1="16.9" x2="32.1" y2="17.05" width="0.1" layer="1"/>
+<wire x1="32.1" y1="17.05" x2="32.4" y2="17.05" width="0.1" layer="1"/>
+<wire x1="32.4" y1="17.05" x2="32.4" y2="16.9" width="0.1" layer="1"/>
+<wire x1="32.4" y1="16.9" x2="32.10051875" y2="16.9" width="0.1" layer="1"/>
+<wire x1="32.1" y1="16.9" x2="32.10051875" y2="16.9" width="0.1" layer="1"/>
+<wire x1="32.10051875" y1="16.9" x2="32.10051875" y2="16.976090625" width="0.1" layer="1"/>
+<wire x1="32.10051875" y1="16.976090625" x2="32.397065625" y2="16.976090625" width="0.1" layer="1"/>
+<wire x1="32.397065625" y1="16.976090625" x2="32.397065625" y2="16.97355" width="0.1" layer="1"/>
+</signal>
+<signal name="S$34">
+<wire x1="31.816675" y1="16.437609375" x2="31.892875" y2="16.437609375" width="0.1" layer="1"/>
+<wire x1="31.892875" y1="16.437609375" x2="31.892875" y2="16.47698125" width="0.1" layer="1"/>
+<wire x1="31.892875" y1="16.47698125" x2="32.40214375" y2="16.47698125" width="0.1" layer="1"/>
+<wire x1="32.40214375" y1="16.47698125" x2="32.40214375" y2="16.742409375" width="0.1" layer="1"/>
+<wire x1="32.40214375" y1="16.742409375" x2="32.273875" y2="16.742409375" width="0.1" layer="1"/>
+<wire x1="32.273875" y1="16.742409375" x2="32.273875" y2="16.73986875" width="0.1" layer="1"/>
+<wire x1="32.273875" y1="16.73986875" x2="32.26561875" y2="16.73986875" width="0.1" layer="1"/>
+<wire x1="32.26561875" y1="16.73986875" x2="32.26561875" y2="16.497934375" width="0.1" layer="1"/>
+<wire x1="32.26561875" y1="16.497934375" x2="32.331659375" y2="16.497934375" width="0.1" layer="1"/>
+<wire x1="32.331659375" y1="16.497934375" x2="32.331659375" y2="16.67383125" width="0.1" layer="1"/>
+</signal>
 </signals>
